File: poe.kicad_sch (KiCad schematic)
At the start: 42 parts, among them J3 7498210002, U4 Oscillator_3225, U5 LAN8720A, U6 SPBW03G-05, U7 TPS2375-1

Commit message: updated files
Parts:
- R10, R11, R12: value 33 -> 20
- R13, R14, R15, R16: value 10 -> 20
Other:
- note added: "Increase cap size a lot, wtf jana"
- note added: "MDIO pullup"
- note added: "RXER to IO13 + pullup"
- note added: "to 10k or 5k1, because strapping pins"
- note added: "to VDDA"
Changed lines of the file:
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@@
     (stroke (width 0) (type default) (color 0 0 0 0))
+  )
+  (text "RXER to IO13 + pullup" (at 24.13 97.79 0)
+    (effects (font (size 1.27 1.27)) (justify left bottom))
+  )
+  (text "to VDDA\n" (at 116.84 78.74 0)
+    (effects (font (size 1.27 1.27)) (justify left bottom))
+  )
+  (text "Increase cap size a lot, wtf jana" (at 158.75 135.89 0)
+    (effects (font (size 1.27 1.27)) (justify left bottom))
+  )
+  (text "MDIO pullup\n" (at 39.37 105.41 0)
+    (effects (font (size 1.27 1.27)) (justify left bottom))
+  )
+  (text "to 10k or 5k1, because strapping pins" (at 96.52 116.84 0)
+    (effects (font (size 1.27 1.27)) (justify left bottom))
+  )
+  (text "to VDDA" (at 227.33 68.58 0)
+    (effects (font (size 1.27 1.27)) (justify left bottom))
   )
   (label "LED_Y" (at 120.65 111.76 0)
@@
     (in_bom yes) (on_board yes)
     (property "Reference" "R12" (id 0) (at 67.31 121.92 90))
-    (property "Value" "33" (id 1) (at 67.31 119.38 90))
+    (property "Value" "20" (id 1) (at 67.31 119.38 90))
     (property "Footprint" "otter:R_0402" (id 2) (at 67.31 119.38 0)
       (effects (font (size 1.27 1.27)) hide)
@@
     (in_bom yes) (on_board yes)
     (property "Reference" "R16" (id 0) (at 64.77 100.33 90))
-    (property "Value" "10" (id 1) (at 68.58 101.6 90))
+    (property "Value" "20" (id 1) (at 68.58 101.6 90))
     (property "Footprint" "otter:R_0402" (id 2) (at 68.58 101.6 0)
       (effects (font (size 1.27 1.27)) hide)
@@
     (in_bom yes) (on_board yes)
     (property "Reference" "R14" (id 0) (at 64.77 95.25 90))
-    (property "Value" "10" (id 1) (at 68.58 96.52 90))
+    (property "Value" "20" (id 1) (at 68.58 96.52 90))
     (property "Footprint" "otter:R_0402" (id 2) (at 68.58 96.52 0)
       (effects (font (size 1.27 1.27)) hide)
@@
     (in_bom yes) (on_board yes)
     (property "Reference" "R13" (id 0) (at 64.77 92.71 90))
-    (property "Value" "10" (id 1) (at 68.58 93.98 90))
+    (property "Value" "20" (id 1) (at 68.58 93.98 90))
     (property "Footprint" "otter:R_0402" (id 2) (at 68.58 93.98 0)
       (effects (font (size 1.27 1.27)) hide)
@@
     (in_bom yes) (on_board yes)
     (property "Reference" "R15" (id 0) (at 64.77 97.79 90))
-    (property "Value" "10" (id 1) (at 68.58 99.06 90))
+    (property "Value" "20" (id 1) (at 68.58 99.06 90))
     (property "Footprint" "otter:R_0402" (id 2) (at 68.58 99.06 0)
       (effects (font (size 1.27 1.27)) hide)
@@
     (in_bom yes) (on_board yes)
     (property "Reference" "R10" (id 0) (at 60.96 116.84 90))
-    (property "Value" "33" (id 1) (at 63.5 116.84 90))
+    (property "Value" "20" (id 1) (at 63.5 116.84 90))
     (property "Footprint" "otter:R_0402" (id 2) (at 63.5 116.84 0)
       (effects (font (size 1.27 1.27)) hide)
@@
     (in_bom yes) (on_board yes)
     (property "Reference" "R11" (id 0) (at 67.31 116.84 90))
-    (property "Value" "33" (id 1) (at 67.31 114.3 90))
+    (property "Value" "20" (id 1) (at 67.31 114.3 90))
     (property "Footprint" "otter:R_0402" (id 2) (at 67.31 114.3 0)
       (effects (font (size 1.27 1.27)) hide)

Commit message: updated to V1.1
Parts:
- removed C24: 47uF 100V, otter:C_1812, symbol Device:C_Polarized_Small
- removed C26: 100n, otter:C_0805, symbol Device:C_Small
- removed L1: 4u7, Inductor_SMD:L_1210_3225Metric, symbol Device:L_Small
- removed R28: 100k, otter:R_0402, symbol Device:R_Small
- removed R29: 24k9, otter:R_0402, symbol Device:R_Small
- removed R30: 357, otter:R_0402, symbol Device:R_Small
- removed R31: 178k, otter:R_0402, symbol Device:R_Small
- removed U6: SPBW03G-05, otter:SPBW03G-05, symbol otter:SPBW03G-05
- removed U7: TPS2375-1, Package_SO:TSSOP-8_4.4x3mm_P0.65mm, symbol Regulator_Controller:TPS2375-1
- added C24: 1u, otter:C_0603, symbol Device:C_Small
- added C26: 47uF 35V, otter:C_1812, symbol Device:C_Polarized_Small
- added C32: 100n, otter:C_0805, symbol Device:C_Small
- added R7: DNP, Resistor_SMD:R_1210_3225Metric, symbol Device:R_Small
- added R8: 5k1, otter:R_0402, symbol Device:R_Small
- added U6: AMS1117-5.0, Package_TO_SOT_SMD:SOT-223-3_TabPin2, symbol Regulator_Linear:AMS1117-5.0
- added U7: DP99xx, otter:DP99xx, symbol otter:DP99xx
- R18, R19: value 49R9 -> 10k
- R27: value 20 -> 5k1
Connections:
- net +3V3: now also R27.2, R8.2; no longer C25.2, J3.3 (TX), J3.4 (RX), R15.2, R20.1, R24.1, R25.1, R26.1
- net +5V: now also U6.2 (VO)
- net ETH_MDIO: now also R27.1
- net GND: now also C24.1, C26.2, C32.2, R7.1, U6.1 (GND), U7.3 (VDC-)
- net at D15.2 (A2), J3.9 (V+): now also U7.5 (VIN+), U7.6 (VIN+)
- net at D15.1 (A1), J3.10 (V-): now also U7.7 (VIN-), U7.8 (VIN-)
- net at C10.2, C8.2, FB1.2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: now also C25.2, J3.3 (TX), J3.4 (RX), R20.1, R24.1, R25.1, R26.1
- new net: C24.2, C26.1, C32.1, R7.2, U6.3 (VI), U7.1 (VDC+), U7.2 (VDC+)
- new net ETH_RXER: R15.2, R8.1
- no-connect marks 1 -> 2
Other:
- note added: "CHANGELOG: ADDED ETH_RXER"
- note removed: "Increase cap size a lot, wtf jana"
- note removed: "MDIO pullup"
- note removed: "RXER to IO13 + pullup"
- note removed: "to 10k or 5k1, because strapping pins"
- note removed: "to VDDA"
