File: voc-tally-light.kicad_pcb (KiCad board)
At the start: 2 copper layers, 80 x 80 mm, 97 parts, among them J1 USB, J2 M3, J3 7498210002, Q1 BC857, Q2 BC857, Q3 2N7002, SW2 Mode, SW3 Brightness, U1 otter_USBLC6-4, U2 ESP32-WROOM-32U, U3 CH340G, U4 Oscillator_3225, U5 LAN8720A, U6 SPBW03G-05, U7 TPS2375-1, U8 AP2204R-3.3, Y1 12Mhz

Commit message: updated files
Parts:
- Q1, Q2: value BC857 -> BC817
- R10, R11, R12: value 33 -> 20
- R13, R14, R15, R16: value 10 -> 20
- moved R5 3.50 mm to (79.2, 113.8), turned to 0 degrees
Connections:
- Q1 pad 1: Net-(Q1-Pad1) -> Net-(R5-Pad1)
- Q1 pad 2: Net-(Q1-Pad2) -> Net-(R6-Pad2)
- Q2 pad 1: Net-(Q1-Pad2) -> Net-(R6-Pad1)
- Q2 pad 2: Net-(Q1-Pad1) -> Net-(R5-Pad2)
- R5 pad 1: Net-(Q1-Pad1) -> Net-(R5-Pad1)
- R6 pad 1: Net-(Q1-Pad2) -> Net-(R6-Pad1)
Routing:
- net Net-(Q1-Pad2): track 5.96 -> 0.00 mm
- net Net-(R6-Pad2): track 10.9 -> 16.4 mm, vias 2 -> 4
- net Net-(R5-Pad2): track 10.7 -> 15.5 mm
- net Net-(Q1-Pad1): track 4.56 -> 0.00 mm
- net Net-(R6-Pad1): track 0.00 -> 3.94 mm
- net Net-(R5-Pad1): track 0.00 -> 2.03 mm
- net GND: vias 188 -> 187

Commit message: updated to V1.1
Parts:
- removed L1: 4u7, Inductor_SMD:L_1210_3225Metric
- removed R28: 100k, otter:R_0402
- removed R29: 24k9, otter:R_0402
- removed R30: 357, otter:R_0402
- removed R31: 178k, otter:R_0402
- added C32: 100n, otter:C_0805, B.Cu at (134.4, 88.5)
- added C33: 1u, otter:C_0603, B.Cu at (119.5, 71.0)
- added P1: TC2030-CTX-Tag-Connect-ESP32, otter:TC2030, B.Cu at (81.0, 109.7)
- added R7: DNP, Resistor_SMD:R_1210_3225Metric, B.Cu at (137.1, 98.9)
- added R8: 5k1, otter:R_0402, B.Cu at (115.0, 84.4)
- C24: value 47uF 100V -> 1u; footprint otter:C_1812 -> otter:C_0603
- C26: value 100n -> 47uF 35V; footprint otter:C_0805 -> otter:C_1812
- Q1, Q2: value BC817 -> S8050
- R18, R19: value 49R9 -> 10k
- R27: value 20 -> 5k1
- U6: value SPBW03G-05 -> AMS1117-5.0; footprint otter:SPBW03G-05 -> Package_TO_SOT_SMD:SOT-223-3_TabPin2
- U7: value TPS2375-1 -> DP99xx; footprint Package_SO:TSSOP-8_4.4x3mm_P0.65mm -> otter:DP99xx
- moved G*** 59.0 mm to (99.8, 132.2), turned to -168 degrees
- moved C24 35.6 mm to (125.5, 77.2), turned to 0 degrees
- moved R27 31.0 mm to (103.7, 86.1)
- moved C26 29.3 mm to (129.8, 86.9), turned to -7 degrees
- moved C23 16.8 mm to (122.0, 77.2), turned to 0 degrees
- moved U6 15.5 mm to (123.5, 82.4), turned to -90 degrees
- moved C30 12.3 mm to (118.0, 76.4), turned to 0 degrees
- moved U7 11.5 mm to (127.9, 99.5), turned to -97 degrees
- moved U8 7.93 mm to (117.2, 79.6), turned to 180 degrees
- moved D15 7.11 mm to (122.0, 111.6), turned to 180 degrees
- moved C31 3.26 mm to (118.2, 82.8), turned to 0 degrees
- moved FB1 1.21 mm to (118.0, 97.3), turned to 180 degrees
Connections:
- C24 pad 1: Net-(C24-Pad1) -> GND
- C25 pad 2: +3V3 -> Net-(C10-Pad2)
- C26 pad 1: Net-(C24-Pad1) -> Net-(C24-Pad2)
- C26 pad 2: Net-(C26-Pad2) -> GND
- D15 pad 1: Net-(C26-Pad2) -> Net-(D15-Pad1)
- D15 pad 2: Net-(C24-Pad1) -> Net-(D15-Pad2)
- J3 pad 10: Net-(C26-Pad2) -> Net-(D15-Pad1)
- J3 pad 3: +3V3 -> Net-(C10-Pad2)
- J3 pad 4: +3V3 -> Net-(C10-Pad2)
- J3 pad 9: Net-(C24-Pad1) -> Net-(D15-Pad2)
- R15 pad 2: +3V3 -> /ETH_RXER
- R20 pad 1: +3V3 -> Net-(C10-Pad2)
- R24 pad 1: +3V3 -> Net-(C10-Pad2)
- R25 pad 1: +3V3 -> Net-(C10-Pad2)
- R26 pad 1: +3V3 -> Net-(C10-Pad2)
- R27 pad 1: Net-(R27-Pad1) -> /ETH_MDIO
- R27 pad 2: Net-(R27-Pad2) -> +3V3
- U2 pad 16: unconnected-(U2-Pad16) -> /ETH_RXER
- U6 pad 1: Net-(C24-Pad2) -> GND
- U6 pad 2: Net-(L1-Pad2) -> +5V
- U6 pad 3: Net-(R27-Pad1) -> Net-(C24-Pad2)
- U7 pad 1: Net-(R31-Pad1) -> Net-(C24-Pad2)
- U7 pad 2: Net-(R30-Pad1) -> Net-(C24-Pad2)
- U7 pad 3: Net-(R29-Pad2) -> GND
- U7 pad 4: Net-(C26-Pad2) -> unconnected-(U7-Pad4)
- U7 pad 5: Net-(C24-Pad2) -> Net-(D15-Pad2)
- U7 pad 6: Net-(R27-Pad2) -> Net-(D15-Pad2)
- U7 pad 7: unconnected-(U7-Pad7) -> Net-(D15-Pad1)
- U7 pad 8: Net-(C24-Pad1) -> Net-(D15-Pad1)
Routing:
- net Net-(D15-Pad1): track 0.00 -> 48.0 mm
- net Net-(C24-Pad1): track 42.5 -> 0.00 mm
- net Net-(C26-Pad2): track 36.1 -> 0.00 mm
- net Net-(C10-Pad2): track 9.62 -> 44.9 mm, vias 2 -> 5
- net Net-(C24-Pad2): track 0.00 -> 27.1 mm
- net Net-(D15-Pad2): track 0.00 -> 26.4 mm
- net /ETH_RXER: track 0.00 -> 19.6 mm, vias 0 -> 2
- net +3V3: track 224.4 -> 235.3 mm, vias 12 -> 7
- net Net-(L1-Pad2): track 7.53 -> 0.00 mm
- net EN: track 58.9 -> 66.3 mm, vias 2 -> 4
- net Net-(R27-Pad1): track 5.57 -> 0.00 mm
- net TXD: track 47.5 -> 52.7 mm, vias 0 -> 2
- net IO0: track 79.1 -> 84.2 mm
- net +5V: track 386.7 -> 382.1 mm, vias 5 -> 6
- net Net-(R29-Pad2): track 3.95 -> 0.00 mm
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- removed copper zone on B.Cu, net Net-(C24-Pad2)
- removed copper zone on B.Cu, net Net-(C26-Pad2)
Other:
- board text added: "@_Jana_Marie 2022 v1.1"
- board text removed: "@_Jana_Marie 2022 v1.0"
