File: voc-tally-light.kicad_sch (KiCad schematic)
At the start: 26 parts, among them J1 USB, J2 M3, Q1 BC857, Q2 BC857, SW2 Mode, SW3 Brightness, U1 otter_USBLC6-4, U2 ESP32-WROOM-32U, U3 CH340G, U8 AP2204R-3.3, Y1 12Mhz

Commit message: updated files
Parts:
- removed Q1, Q2: BC857, Package_TO_SOT_SMD:SOT-23, symbol Transistor_BJT:BC857
- added Q? (x2): S8050, Package_TO_SOT_SMD:SOT-23, symbol Transistor_BJT:BC847
Connections:
- net EN: now also Q?.3 (C)
- net IO0: now also Q?.3 (C)
- net at R5.1: now also Q?.1 (B)
- net at R6.1: now also Q?.1 (B)
- net at R5.2, U3.13 (~{DTR}): now also Q?.2 (E)
- net at R6.2, U3.14 (~{RTS}): now also Q?.2 (E)
Other:
- moved on the sheet: R5, R6

Commit message: updated to V1.1
Parts:
- added P1: TC2030-CTX-Tag-Connect-ESP32, otter:TC2030, symbol otter:TC2030-CTX-Tag-Connect-ESP32
- gave numbers to parts that had none: 2
Connections:
- net EN: now also P1.6 (EN)
- net GND: now also P1.5 (GND)
- net IO0: now also P1.2 (IO0)
- net RXD: now also P1.4 (RXD)
- net TXD: now also P1.3 (TXD)
- net ETH_RXER: now reaches U2.16 (IO13)
- no-connect marks 9 -> 10
Other:
- sheet ETH ports: added ETH_RXER; removed none
- note removed: "PoE 802.3af DONE LEDs DONE Programmer DONE 3/4" Schraube KINDA DONE 2 x input switch DONE Ethernet DONE Parts on bottom side winkekatze on top DONE Power over Estrogen"
